File: Hardware/Fairybox.kicad_sch (KiCad schematic)
At the start: 83 parts, among them J1 REED, J2 BATTERY, J3 CHARGE_BOARD, Q1 SI2302, Q10 C114, Q2 C114, Q3 C114, Q4 C114, Q5 C114, Q6 C114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

Commit message: I forget
Parts:
- added D10: BLUE, Diode_SMD:D_1206_3216Metric, symbol Device:LED_Small_Filled
- added D11: RED, Diode_SMD:D_1206_3216Metric, symbol Device:LED_Small_Filled
- added Q11, Q12: SI2302, Package_TO_SOT_SMD:SOT-23, symbol Transistor_FET:TSM2302CX
- added R18, R23: 470R, Resistor_SMD:R_1206_3216Metric, symbol Device:R_Small
Connections:
- net +5V: now also R18.1, R23.1
- net GND: now also D11.1 (K), Q11.2 (S), Q12.2 (S)
- new net: D11.2 (A), Q12.3 (D), R23.2
- new net: Q11.1 (G), Q12.1 (G)
- new net: D10.1 (K), Q11.3 (D)
- new net: D10.2 (A), R18.2
