File: Hardware/Fairybox.kicad_pcb (KiCad board)
At the start: 2 copper layers, 91.4 x 54.1 mm, 73 parts, among them J1 REED, J2 JST B4B-PH-K-S, Q1 locked, Q10 locked, Q2 locked, Q3 locked, Q4 locked, Q5 locked, Q6 locked, Q7 locked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

Commit message: many
Parts:
- added Q14: AO3401A, Package_TO_SOT_SMD:SOT-23, F.Cu at (82.5, 59.7)
- added Q15: SI2302, Package_TO_SOT_SMD:SOT-23, F.Cu at (90.2, 64.8)
- added Q16: SI2302, Package_TO_SOT_SMD:SOT-23, F.Cu at (77.5, 61.0)
- added R20: 100K, Resistor_SMD:R_1206_3216Metric, F.Cu at (55.9, 75.6)
- added R22: 1M, Resistor_SMD:R_1206_3216Metric, F.Cu at (47.0, 62.2)
- added R23: 330k, Resistor_SMD:R_1206_3216Metric, F.Cu at (38.1, 58.4)
- D4: value locked -> RED
- R18, R19, R7: value 220R -> 470R
- R6: value 1K -> 10K
- moved JP4 30.1 mm to (151.4, 96.5)
- moved JP6 27.6 mm to (83.8, 126.0)
- moved JP2 24.6 mm to (79.8, 122.9)
- moved JP8 22.1 mm to (148.8, 97.5)
- moved JP7 13.1 mm to (149.9, 99.6)
- moved JP1 8.47 mm to (81.3, 69.1)
- moved R6 8.26 mm to (53.3, 85.1)
- moved JP5 6.16 mm to (79.8, 69.1)
- moved D25 6.10 mm to (63.5, 83.8)
- moved U2 5.78 mm to (53.3, 80.0), turned to 0 degrees
- moved J2 5.75 mm to (54.9, 59.5), turned to -90 degrees
- moved R16 4.28 mm to (63.5, 78.7)
- moved Q1 2.69 mm to (56.2, 71.5)
- moved CE1 0.31 mm to (56.9, 89.8)
- moved R15 0.13 mm to (134.4, 75.2)
Connections:
- net /Q1_BASE renamed /Q1_GATE
- R10 pad 1: +5V -> /BLUE LED RESISTOR ANODES
- R11 pad 1: +5V -> /BLUE LED RESISTOR ANODES
- R14 pad 1: +5V -> /+5V B-LED
- R15 pad 1: +5V -> /+5V B-LED
- R2 pad 1: +5V -> /+5V B-LED
- R4 pad 1: +5V -> /+5V B-LED
- R8 pad 1: +5V -> /+5V B-LED
- R9 pad 1: +5V -> /+5V B-LED
Routing:
- net /CHARGE BOARD OUT B+: track 45.6 -> 25.6 mm
- net GND: track 20.8 -> 1.66 mm, vias 1 -> 3
- net /Q1_GATE: track 3.36 -> 21.9 mm, vias 0 -> 2
- net +5V: track 135.7 -> 122.4 mm
- net /REED_RETURN: track 23.7 -> 15.1 mm
- net /LI-ION_POS: track 14.2 -> 7.75 mm
- net /Q6_COL: track 23.0 -> 29.2 mm
- net /Q2_COL: track 22.1 -> 28.2 mm
- net /LI-ION_NEG: track 84.4 -> 87.2 mm
- net /D9_AN: track 2.19 -> 4.68 mm
- net /D25_AN: track 4.05 -> 2.22 mm
- net /D20_AN: track 9.31 -> 8.68 mm
- added copper zone on F.Cu, net /CHARGE BOARD OUT B+
- added copper zone on F.Cu, net /CHARGE BOARD OUT B-
- added copper zone on F.Cu, net GND

Commit message: a lot
Parts:
- added BAT1: locked, Battery:18650 battery sled 1x, F.Cu at (62.2, 61.7)
- R22, R23: moved to B.Cu
- TP1: value locked -> RST
- TP3: value locked -> MISO
- TP4: value locked -> MOSI
- TP5: value locked -> VCC
- U1: value locked -> ATTINY85
- moved JP2 51.7 mm to (64.0, 73.7)
- moved R23 30.2 mm to (65.5, 71.1), turned to -90 degrees
- moved Q14 28.3 mm to (59.4, 75.9)
- moved Q15 22.0 mm to (71.1, 75.9), turned to 90 degrees
- moved Q16 19.9 mm to (64.4, 75.9)
- moved JP1 19.3 mm to (62.0, 68.3)
- moved R22 18.3 mm to (63.0, 71.1), turned to 90 degrees
- moved JP9 16.8 mm to (62.0, 73.7)
- moved JP5 15.8 mm to (64.0, 68.3)
- moved D25 4.95 mm to (63.5, 88.8)
- moved JP3 4.75 mm to (52.1, 81.7)
- moved D9 4.39 mm to (119.0, 80.8)
- moved R1 4.13 mm to (71.1, 80.0)
- moved R14 3.08 mm to (126.5, 77.7)
- moved TP12 3.05 mm to (137.2, 98.4)
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Connections:
- net /5 renamed /PB0 PHY
- net /6 renamed /PB1 PHY
- net /7 renamed /PB2 PHY
- net Net-(Q14-Pad1) renamed /LBAT_NOT
- net Net-(Q14-Pad3) renamed /Q15_COL
- J1 pad 1: /CHARGE BOARD OUT B+ -> /REED_IN
- J1 pad 2: /REED_RETURN -> /Q1_GATE
- R10 pad 1: /BLUE LED RESISTOR ANODES -> /+5V B-LED
- R11 pad 1: /BLUE LED RESISTOR ANODES -> /+5V B-LED
- R6 pad 1: /REED_RETURN -> /REED_IN
- R6 pad 2: /Q1_GATE -> /CHARGE BOARD OUT B+
- R8 pad 1: /+5V B-LED -> +5V
Routing:
- net /+5V B-LED: track 0.00 -> 70.8 mm
- net +5V: track 122.4 -> 153.4 mm
- net /REED_IN: track 0.00 -> 21.3 mm
- net /CHARGE BOARD OUT B-: track 0.00 -> 16.4 mm
- net /REED_RETURN: track 15.1 -> 0.00 mm
- net /D6_AN: track 33.1 -> 18.3 mm
- net /Q1_GATE: track 21.9 -> 36.7 mm
- net /Q2_COL: track 28.2 -> 15.2 mm
- net /Q4_COL: track 32.1 -> 19.2 mm
- net /Q15_COL: track 0.00 -> 10.2 mm
- net /LBAT_NOT: track 0.00 -> 9.71 mm, vias 0 -> 1
- net /LI-ION_POS: track 7.75 -> 13.8 mm, vias 0 -> 1
- net /Q6_COL: track 29.2 -> 25.3 mm
- net /CHARGE BOARD OUT B+: track 25.6 -> 21.8 mm
- net /MCU GPIO4: track 112.5 -> 109.1 mm
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- removed copper zone on F.Cu, net /CHARGE BOARD OUT B+
- removed copper zone on F.Cu, net /CHARGE BOARD OUT B-
- removed copper zone on F.Cu, net GND
Other:
- board text added: "8"
- board text added: "AND"
- board text added: "MISO"
- board text added: "MOSI"
- board text added: "NOT"
- board text added: "SCK"
- board text removed: "5V"
- board text removed: "6"
- board text removed: "B+"
- board text removed: "B-"

Commit message: Edge cut.
Parts:
- moved R23 0.38 mm to (65.9, 71.1)
Changed lines of the file:
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@@
     (pad_to_mask_clearance 0)
     (solder_mask_min_width 0.12)
-    (aux_axis_origin 129.032 50.8)
+    (aux_axis_origin 50.8 50.8)
+    (grid_origin 50.8 50.8)
     (pcbplotparams
       (layerselection 0x00010fc_ffffffff)
@@
   )
   (footprint "Resistor_SMD:R_1206_3216Metric" (layer "B.Cu")
-    (at 65.532 71.12 -90)
+    (at 65.913 71.12 -90)
     (descr "Resistor SMD 1206 (3216 Metric), square (rectangular) end terminal, IPC_7351 nominal, (Body size source: IPC-SM-782 page 72, https://www.pcb-3d.com/wordpress/wp-content/uploads/ipc-sm-782a_amendment_1_and_2.pdf), generated with kicad-footprint-generator")
     (tags "resistor")
@@
     )
   )
+  (gr_line (start 119.8 107.8) (end 144.8 107.8) (layer "F.Cu") (width 0.254))
+  (gr_line (start 144.8 50.8) (end 50.8 50.8) (layer "F.Cu") (width 0.254))
+  (gr_line (start 144.8 107.8) (end 144.8 50.8) (layer "F.Cu") (width 0.254))
+  (gr_line (start 50.8 107.8) (end 75.8 107.8) (layer "F.Cu") (width 0.254))
+  (gr_line (start 75.8 107.8) (end 75.8 100.8) (layer "F.Cu") (width 0.254))
+  (gr_line (start 119.8 100.8) (end 119.8 107.8) (layer "F.Cu") (width 0.254))
+  (gr_line (start 50.8 50.8) (end 50.8 107.8) (layer "F.Cu") (width 0.254))
+  (gr_line (start 75.8 100.8) (end 119.8 100.8) (layer "F.Cu") (width 0.254))
   (gr_rect (start 121.8438 118.4148) (end 80.137 111.8108) (layer "B.SilkS") (width 0.254) (fill none))
   (gr_line (start 127.59 96.95) (end 139.07 96.95) (layer "F.SilkS") (width 0.15))
@@
   (segment (start 80.01 77.724) (end 87.63 77.724) (width 0.508) (layer "F.Cu") (net 5))
   (segment (start 93.98 73.914) (end 94.488 74.422) (width 0.508) (layer "F.Cu") (net 5))
-  (segment (start 84.92625 87.72025) (end 84.92625 90.33375) (width 0.508) (layer "F.Cu") (net 6))
   (segment (start 81.28 98.425) (end 81.28 95.25) (width 0.2) (layer "F.Cu") (net 6))
-  (segment (start 80.01 82.804) (end 84.92625 87.72025) (width 0.508) (layer "F.Cu") (net 6))
-  (segment (start 84.92625 90.33375) (end 81.28 93.98) (width 0.508) (layer "F.Cu") (net 6))
-  (segment (start 81.28 93.98) (end 81.28 95.25) (width 0.508) (layer "F.Cu") (net 6))
+  (segment (start 81.28 94.107) (end 81.28 95.25) (width 0.508) (layer "F.Cu") (net 6))
+  (segment (start 84.963 87.757) (end 84.963 90.424) (width 0.508) (layer "F.Cu") (net 6))
+  (segment (start 84.963 90.424) (end 81.28 94.107) (width 0.508) (layer "F.Cu") (net 6))
+  (segment (start 80.01 82.804) (end 84.963 87.757) (width 0.508) (layer "F.Cu") (net 6))
   (segment (start 67.31 87.63) (end 67.31 84.587) (width 0.6) (layer "F.Cu") (net 7))
   (segment (start 69.601 82.047) (end 71.12 83.566) (width 0.508) (layer "F.Cu") (net 8))
@@
   (segment (start 133.641665 86.068335) (end 133.762625 85.947375) (width 0.508) (layer "F.Cu") (net 14))
   (segment (start 131.101665 88.9) (end 131.101665 89.979935) (width 0.508) (layer "F.Cu") (net 15))
-  (segment (start 124.4246 91.4654) (end 120.64 95.25) (width 0.508) (layer "F.Cu") (net 15))
-  (segment (start 127.4826 91.4654) (end 128.016 90.932) (width 0.508) (layer "F.Cu") (net 15))
+  (segment (start 120.64 95.25) (end 124.2468 91.6432) (width 0.508) (layer "F.Cu") (net 15))
+  (segment (start 124.2468 91.6432) (end 127.3048 91.6432) (width 0.508) (layer "F.Cu") (net 15))
+  (segment (start 127.3048 91.6432) (end 128.016 90.932) (width 0.508) (layer "F.Cu") (net 15))
   (segment (start 131.101665 89.979935) (end 129.54 91.5416) (width 0.508) (layer "F.Cu") (net 15))
-  (segment (start 124.4246 91.4654) (end 127.4826 91.4654) (width 0.508) (layer "F.Cu") (net 15))
   (segment (start 129.54 91.5416) (end 127.3302 91.5416) (width 0.508) (layer "F.Cu") (net 15))
-  (segment (start 128.016 90.932) (end 128.016 89.5664) (width 0.508) (layer "F.Cu") (net 15))
   (segment (start 120.64 98.796) (end 120.64 95.25) (width 0.15) (layer "F.Cu") (net 15))
+  (segment (start 128.016 90.932) (end 128.016 89.5664) (width 0.508) (layer "F.Cu") (net 15))
   (segment (start 54.9656 99.822) (end 52.07 99.822) (width 0.1524) (layer "F.Cu") (net 16))
   (segment (start 51.816 99.568) (end 51.816 87.503) (width 0.1524) (layer "F.Cu") (net 16))
@@
   (segment (start 111.506 84.582) (end 111.506 82.804) (width 0.508) (layer "F.Cu") (net 19))
   (segment (start 113.3793 88.699967) (end 113.3793 86.4553) (width 0.508) (layer "F.Cu") (net 19))
-  (segment (start 127.3556 93.4212) (end 133.0452 93.4212) (width 0.508) (layer "F.Cu") (net 20))
-  (segment (start 134.3914 93.345) (end 134.493 93.4466) (width 0.508) (layer "F.Cu") (net 20))
-  (segment (start 135.587822 93.4466) (end 135.613222 93.4212) (width 0.508) (layer "F.Cu") (net 20))
+  (segment (start 129.794 93.5736) (end 132.8928 93.5736) (width 0.508) (layer "F.Cu") (net 20))
+  (segment (start 133.2738 93.1926) (end 135.384622 93.1926) (width 0.508) (layer "F.Cu") (net 20))
   (segment (start 137.16 95.25) (end 137.16 98.425) (width 0.508) (layer "F.Cu") (net 20))
   (segment (start 126.99 93.7868) (end 127.3556 93.4212) (width 0.508) (layer "F.Cu") (net 20))
-  (segment (start 133.1214 93.345) (end 134.3914 93.345) (width 0.508) (layer "F.Cu") (net 20))
-  (segment (start 134.493 93.4466) (end 135.587822 93.4466) (width 0.508) (layer "F.Cu") (net 20))
-  (segment (start 135.613222 93.4212) (end 137.16 94.967978) (width 0.508) (layer "F.Cu") (net 20))
+  (segment (start 132.8928 93.5736) (end 133.2738 93.1926) (width 0.508) (layer "F.Cu") (net 20))
+  (segment (start 127.3556 93.4212) (end 129.6416 93.4212) (width 0.508) (layer "F.Cu") (net 20))
+  (segment (start 135.384622 93.1926) (end 137.16 94.967978) (width 0.508) (layer "F.Cu") (net 20))
   (segment (start 126.99 95.25) (end 126.99 93.7868) (width 0.508) (layer "F.Cu") (net 20))
-  (segment (start 133.0452 93.4212) (end 133.1214 93.345) (width 0.508) (layer "F.Cu") (net 20))
+  (segment (start 129.6416 93.4212) (end 129.794 93.5736) (width 0.508) (layer "F.Cu") (net 20))
   (segment (start 83.566 81.788) (end 84.836 83.058) (width 0.508) (layer "F.Cu") (net 21))
   (segment (start 83.566 80.01) (end 83.566 81.788) (width 0.508) (layer "F.Cu") (net 21))
@@
   (segment (start 51.499661 80.264) (end 51.499661 79.056339) (width 0.1524) (layer "B.Cu") (net 40))
   (segment (start 51.499661 79.056339) (end 52.832 77.724) (width 0.1524) (layer "B.Cu") (net 40))
+  (segment (start 91.44 70.612) (end 93.472 70.612) (width 0.508) (layer "F.Cu") (net 41))
   (segment (start 107.823 77.724) (end 111.474375 77.724) (width 0.508) (layer "F.Cu") (net 41))
+  (segment (start 106.2482 71.1962) (end 107.815 72.763) (width 0.508) (layer "F.Cu") (net 41))
+  (segment (start 100.3554 71.1962) (end 106.2482 71.1962) (width 0.508) (layer "F.Cu") (net 41))
   (segment (start 93.6498 70.7898) (end 98.1202 70.7898) (width 0.508) (layer "F.Cu") (net 41))
-  (segment (start 107.815 72.763) (end 107.815 76.962) (width 0.508) (layer "F.Cu") (net 41))
-  (segment (start 91.2622 70.7898) (end 91.44 70.612) (width 0.508) (layer "F.Cu") (net 41))
   (segment (start 85.4202 70.7898) (end 91.2622 70.7898) (width 0.508) (layer "F.Cu") (net 41))
   (segment (start 93.472 70.612) (end 93.6498 70.7898) (width 0.508) (layer "F.Cu") (net 41))
-  (segment (start 100.3554 70.8914) (end 105.9434 70.8914) (width 0.508) (layer "F.Cu") (net 41))
-  (segment (start 98.298 70.612) (end 100.076 70.612) (width 0.508) (layer "F.Cu") (net 41))
-  (segment (start 105.9434 70.8914) (end 107.815 72.763) (width 0.508) (layer "F.Cu") (net 41))
-  (segment (start 98.1202 70.7898) (end 98.298 70.612) (width 0.508) (layer "F.Cu") (net 41))
   (segment (start 75.946 74.93) (end 83.566 74.93) (width 0.508) (layer "F.Cu") (net 41))
-  (segment (start 100.076 70.612) (end 100.3554 70.8914) (width 0.508) (layer "F.Cu") (net 41))
   (segment (start 74.676 74.93) (end 75.946 74.93) (width 0.508) (layer "F.Cu") (net 41))
-  (segment (start 83.566 72.644) (end 85.4202 70.7898) (width 0.508) (layer "F.Cu") (net 41))
-  (segment (start 91.44 70.612) (end 93.472 70.612) (width 0.508) (layer "F.Cu") (net 41))
+  (segment (start 83.566 74.93) (end 83.566 72.644) (width 0.508) (layer "F.Cu") (net 41))
+  (segment (start 107.815 72.763) (end 107.815 76.962) (width 0.508) (layer "F.Cu") (net 41))
   (segment (start 111.474375 77.724) (end 115.19575 77.724) (width 0.508) (layer "F.Cu") (net 41))
   (segment (start 72.801 76.805) (end 74.676 74.93) (width 0.508) (layer "F.Cu") (net 41))
+  (segment (start 91.2622 70.7898) (end 91.44 70.612) (width 0.508) (layer "F.Cu") (net 41))
+  (segment (start 83.566 72.644) (end 85.4202 70.7898) (width 0.508) (layer "F.Cu") (net 41))
   (segment (start 126.459875 77.724) (end 133.762625 77.724) (width 0.508) (layer "F.Cu") (net 41))
-  (segment (start 83.566 74.93) (end 83.566 72.644) (width 0.508) (layer "F.Cu") (net 41))
+  (segment (start 98.1202 70.7898) (end 98.3742 71.0438) (width 0.508) (layer "F.Cu") (net 41))
+  (segment (start 100.203 71.0438) (end 100.3554 71.1962) (width 0.508) (layer "F.Cu") (net 41))
   (segment (start 115.19575 77.724) (end 126.459875 77.724) (width 0.508) (layer "F.Cu") (net 41))
   (segment (start 72.07 76.805) (end 72.801 76.805) (width 0.508) (layer "F.Cu") (net 41))
+  (segment (start 98.3742 71.0438) (end 100.203 71.0438) (width 0.508) (layer "F.Cu") (net 41))
   (segment (start 58.42 74.996) (end 63.18 74.996) (width 0.1524) (layer "F.Cu") (net 42))
   (segment (start 62.992 74.996) (end 62.992 73.914) (width 0.508) (layer "F.Cu") (net 42))

Commit message: not sure
Parts:
- added CC1: 0.22uF, Capacitor_SMD:C_1206_3216Metric, F.Cu at (94.5, 93.0)
- CC4: footprint Capacitor_THT:C_Disc_D3.0mm_W2.0mm_P2.50mm -> Capacitor_SMD:C_1206_3216Metric
- moved CC4 1.50 mm to (91.2, 80.5)
Connections:
- U1 pad 4: GND -> (no net)
Routing:
- net GND: track 2.80 -> 21.4 mm, vias 2 -> 4
- net /PB0 PHY: track 27.0 -> 32.1 mm
- net /PB1 PHY: track 32.4 -> 36.8 mm
- net /PB2 PHY: track 37.9 -> 40.1 mm
- net /MCU RST: track 20.7 -> 22.5 mm
- net /D3_AN: track 9.83 -> 10.9 mm
- net +5V: track 153.4 -> 154.4 mm
- net /MCU GPIO3: track 34.7 -> 33.9 mm
